File: underdeskv6/underdesk_macropad_pins.brd (EAGLE design)
At the start: 100 x 80 mm, 13 parts

Commit message: Add files via upload
Parts:
- renumbered B1 to MOTHERBOARD, S1 to ROTARY, U$1 to KEY5, U$2 to KEY4, U$3 to KEY3, U$4 to KEY2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
Connections:
- net VDD renamed +5V
Routing:
- net +5V: track 64.2 -> 0.00 mm
Other:
- board text added: "LIVE AND LEARN"
