File: underdeskv6/underdesk_macropad_pins.sch (EAGLE design)
At the start: 13 parts

Commit message: Add files via upload
Parts:
- renumbered B1 to MOTHERBOARD, S1 to ROTARY, U$1 to KEY5, U$2 to KEY4, U$3 to KEY3, U$4 to KEY2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
Connections:
- new net +5V: LED1.VDD, LED2.VDD, LED3.VDD, LED4.VDD, LED5.VDD, LED6.VDD
